File: 1.Hardware/Kicad/E-LCD2/E-LCD2.kicad_pcb (KiCad board)
At the start: 2 copper layers, 58.3 x 36.3 mm, 40 parts, among them J1 USB-C, Q1 S8050, Q2 S8050, Q3 S8050, SW1 Reset, SW2 Key-A, SW3 Key-B, SW4 Key-C, U1 AMS1117-3.3, U2 ESP32-S32MB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

Commit message: PCB done
Other:
- board text added: "Designed By Forairaaaaa"
- board text added: "LCD-2.0-IPS-ST7789-12PIN"
- board text added: "R5"
- board text added: "https://gitee.com/forairaaaaa/e-lcd2.git"
- board text removed: "Designed by Forairaaaaa"
- board text removed: "LCD_2.0IPS_ST7789_12PIN"
- board text removed: "LCD_BL_DIS"
Changed lines of the file:
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@@
     )
   )
-  (gr_line (start 162.9918 70.5358) (end 172.974 70.5358) (layer "B.SilkS") (width 0.254))
+  (gr_line (start 167.940558 70.8152) (end 176.601958 70.8152) (layer "B.SilkS") (width 0.1524))
+  (gr_line (start 168.2242 67.0814) (end 168.2242 70.0278) (layer "B.SilkS") (width 0.1524))
   (gr_arc locked (start 158.344657 62.713657) (mid 158.5976 62.103) (end 159.208257 61.850057) (layer "Edge.Cuts") (width 0.1))
   (gr_arc locked (start 216.6874 97.3074) (mid 216.434457 97.918057) (end 215.8238 98.171) (layer "Edge.Cuts") (width 0.1))
@@
   (gr_line locked (start 158.3436 97.3074) (end 158.344657 62.713657) (layer "Edge.Cuts") (width 0.1))
   (gr_line locked (start 215.8238 98.171) (end 159.2072 98.171) (layer "Edge.Cuts") (width 0.1))
-  (gr_text "Designed by Forairaaaaa" (at 175.1838 67.4116 180) (layer "B.SilkS")
+  (gr_text "Designed By Forairaaaaa" (at 176.5554 67.818 180) (layer "B.SilkS")
     (effects (font (size 0.8128 0.8128) (thickness 0.15) italic) (justify mirror))
   )
@@
     (effects (font (size 0.762 0.762) (thickness 0.1524)) (justify mirror))
   )
-  (gr_text "ESP32-S" (at 200.0504 75.946 180) (layer "B.SilkS")
+  (gr_text "ESP32-S" (at 200.1774 75.9206 180) (layer "B.SilkS")
     (effects (font (size 1 1) (thickness 0.15)) (justify mirror))
   )
@@
     (effects (font (size 1 1) (thickness 0.15)) (justify mirror))
   )
+  (gr_text "https://gitee.com/forairaaaaa/e-lcd2.git" (at 181.896658 69.6214 180) (layer "B.SilkS")
+    (effects (font (size 0.8128 0.8128) (thickness 0.15) italic) (justify mirror))
+  )
   (gr_text "IO12" (at 175.5394 63.2206 180) (layer "B.SilkS")
     (effects (font (size 0.762 0.762) (thickness 0.1524)) (justify mirror))
   )
-  (gr_text "LCD_BL_DIS" (at 170.561 75.5904 180) (layer "B.SilkS")
+  (gr_text "R5" (at 173.9138 75.5396 90) (layer "B.SilkS")
     (effects (font (size 0.762 0.762) (thickness 0.1524)) (justify mirror))
   )
@@
     (effects (font (size 0.762 0.762) (thickness 0.1524)) (justify mirror))
   )
-  (gr_text "E-LCD2" (at 168.0718 72.263 180) (layer "B.SilkS")
-    (effects (font (size 1.778 1.778) (thickness 0.381) italic) (justify mirror))
+  (gr_text "E-LCD2" (at 172.339 72.1614 180) (layer "B.SilkS")
+    (effects (font (size 1.524 1.524) (thickness 0.3048) italic) (justify mirror))
   )
-  (gr_text "LCD_2.0IPS_ST7789_12PIN" (at 211.6074 87.503 90) (layer "F.SilkS")
+  (gr_text "LCD-2.0-IPS-ST7789-12PIN" (at 194.5894 64.1858 180) (layer "F.SilkS")
     (effects (font (size 1 1) (thickness 0.15)))
   )
-  (gr_text "JLCJLCJLCJLC\n" (at 200.9648 96.1136) (layer "F.SilkS")
+  (gr_text "JLCJLCJLCJLC\n" (at 167.64 64.1858 180) (layer "F.SilkS")
     (effects (font (size 0.762 0.762) (thickness 0.1524)))
   )
@@
     )
   )
+  (group "" (id 19a4f767-dc1c-42e6-80bf-577af4534bd6)
+    (members
+      1c4822b7-b616-4b5d-9c9e-f8a52b71861d
+      67a6b916-ca7a-41fc-ae72-435f634ad18a
+    )
+  )
   (group "" (id 7e776479-96d3-4c2b-817d-6ed3da628f08)
     (members
@@
     )
   )
+  (group "" (id bab46f34-8c8a-41f0-bea2-5779a0f6a524)
+    (members
+      7e776479-96d3-4c2b-817d-6ed3da628f08
+      ee94cadf-f076-4d4f-b155-63eea51e1793
+    )
+  )
+  (group "" (id ee94cadf-f076-4d4f-b155-63eea51e1793)
+    (members
+      19a4f767-dc1c-42e6-80bf-577af4534bd6
+      ae491f31-545b-40e0-b8fa-5a42ad2755b6
+    )
+  )
