File: 1.Hardware/Kicad/E-LCD2/E-LCD2.kicad_sch (KiCad schematic)
At the start: 40 parts, among them J1 USB-C, Q1 S8050, Q2 S8050, Q3 S8050, SW1 Reset, SW2 Key-A, SW3 Key-B, SW4 Key-C, U1 AMS1117-3.3, U2 ESP32-S32MB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

Commit message: PCB done
Other:
- note added: "2.0寸 12pin SPI LCD"
- note added: "DC-DC"
- note added: "LCD-PIN-MAP: MOSI: IO19 SCLK: IO18 CS: IO5 DC: IO16 RST: IO17 BL: IO4"
- note added: "PIN-MAP: LED: IO12 Key-A: IO13 Key-B: IO2 Key-C: IO15"
- note added: "R3：短接（0Ω），使能IO17作LCD复位引脚"
- note added: "R4：串联LCD背光，改变阻值以调节LCD背光亮度"
- note added: "R5：短接（0Ω），失能IO4作LCD背光控制引脚"
- note added: "USB-C"
- note added: "USB_TTL 自动下载，CP2102可用CH9102代替"
- note added: "作者：https://space.bilibili.com/35053144"
- note added: "复位"
- note added: "安信可ESP-32S模组"
- note added: "引脚引出：2 x 1x14P 2.54mm 排针"
- note added: "用户LED、按键"
- note added: "项目仓库：https://gitee.com/forairaaaaa/e-lcd2.git"
- moved on the sheet: C1, C2, C3, C4, C5, C6, C7, C8, C9, H1, H2, J1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
